File: pt2322/amp_pt2322_v_1_0.sch (EAGLE design)
At the start: 33 parts, among them U1 PT2322-S

Commit message: Added interface board for 20x4 lcd, improved firmware for 20x4, refactored pt2322 board
Parts:
- C1, C2, C3, C4, C5: device rcl:CPOL-EUE2-5 -> rcl:CPOL-EUSMCB
- C10, C11, C12, C13, C14, C15, C6, C7, C8, C9: device rcl:C-EU025-025X050 -> rcl:C-EUC0805K
- C16: device rcl:CPOL-EUE2.5-7 -> rcl:CPOL-EUSMCB
- R1, R2, R3, R4, R5, R6, R7, R8: device rcl:R-EU_0207/10 -> rcl:R-EU_R0805
